File: OpenBilgeAlarm.kicad_pcb (KiCad board)
At the start: 2 copper layers, 0 parts

Commit message: Throw everything on board, try to route, start solving the mechanical puzzle
Parts:
- added C1: 1u, Capacitors_SMD:C_1210_HandSoldering, F.Cu at (156.0, 84.1)
- added C10: C, Capacitors_SMD:C_0603_HandSoldering, F.Cu at (157.0, 64.0)
- added C2: CP, Capacitors_ThroughHole:CP_Radial_D5.0mm_P2.50mm, B.Cu at (140.6, 87.8)
- added C3: CP, Capacitors_ThroughHole:CP_Radial_D5.0mm_P2.50mm, B.Cu at (193.0, 93.2)
- added C4: 1u, Capacitors_SMD:C_1210_HandSoldering, F.Cu at (191.9, 88.1)
- added C5: C, Capacitors_SMD:C_0603_HandSoldering, F.Cu at (183.6, 100.6)
- added C6: C, Capacitors_SMD:C_0603_HandSoldering, B.Cu at (201.2, 82.5)
- added C7: C, Capacitors_SMD:C_0603_HandSoldering, F.Cu at (115.0, 86.0)
- added C8: C, Capacitors_SMD:C_0603_HandSoldering, B.Cu at (201.2, 78.8)
- added C9: C, Capacitors_SMD:C_0603_HandSoldering, B.Cu at (212.8, 80.4)
- added D1: 48V, Diodes_SMD:Diode-SMB_Handsoldering, F.Cu at (156.3, 87.8)
- added D10: D_TVS, Diodes_SMD:SOD-323, B.Cu at (211.2, 80.5)
- added D2: D_TVS, Diodes_SMD:SOD-323, F.Cu at (189.6, 91.1)
- added D3: 24V, Diodes_SMD:Diode-SMA_Handsoldering, F.Cu at (148.0, 91.2)
- added D4: 16V, Diodes_SMD:D_SOD-323_HandSoldering, F.Cu at (138.1, 83.0)
- added D5: LED_ARGB, LEDs:LED_D5.0mm-4, F.Cu at (206.5, 56.9)
- added D6: LED, LEDs:LED_D5.0mm, F.Cu at (106.5, 59.0)
- added D7: D_TVS, Diodes_SMD:SOD-323, B.Cu at (199.5, 79.0)
- added D8: D_TVS, Diodes_SMD:SOD-323, F.Cu at (113.0, 86.0)
- added D9: D_TVS, Diodes_SMD:SOD-323, B.Cu at (199.5, 82.0)
- added DS1: LCD16X2, Displays:WC1602A, F.Cu at (123.5, 53.0)
- added F1: Polyfuse, Resistors_THT:R_Box_L8.4mm_W2.5mm_P5.08mm, B.Cu at (187.0, 83.0)
- added J1: CONN_01X02, smalsiukas-footpints:TerminalBlock_5.08-2pol, B.Cu at (154.5, 92.0)
- added J2: CONN_01X04, smalsiukas-footpints:TerminalBlock_5.08-5pol, B.Cu at (166.8, 92.0)
- added LS1: Speaker_Crystal, Buzzer_12x9.5RM7.6, F.Cu at (107.6, 70.0)
- added MK1: Mounting_Hole, Mounting_Holes:MountingHole_3.2mm_M3, F.Cu at (211.5, 91.5)
- added MK2: Mounting_Hole, Mounting_Holes:MountingHole_3.2mm_M3, F.Cu at (103.5, 91.5)
- added MK3: Mounting_Hole, Mounting_Holes:MountingHole_3.2mm_M3, F.Cu at (103.5, 53.5)
- added MK4: Mounting_Hole, Mounting_Holes:MountingHole_3.2mm_M3, F.Cu at (211.5, 53.5)
- added Q1: Q_NMOS_GSD, TO_SOT_Packages_SMD:SOT-23_Handsoldering, F.Cu at (165.0, 54.0)
- added Q2: Q_PMOS_GSD, TO_SOT_Packages_SMD:SOT-23_Handsoldering, F.Cu at (159.7, 59.9)
- added Q3: Q, TO_SOT_Packages_SMD:TO-252-2Lead, F.Cu at (144.9, 82.0)
- added Q4: Q_NMOS_GSD, TO_SOT_Packages_SMD:SOT-23_Handsoldering, F.Cu at (120.0, 70.0)
- added R1: 10R, Resistors_SMD:R_2512, F.Cu at (147.7, 87.9)
- added R10: 330, Resistors_SMD:R_0603_HandSoldering, F.Cu at (173.7, 101.3)
- added R11: 1k, Resistors_SMD:R_0603_HandSoldering, F.Cu at (173.3, 106.4)
- added R12: 330, Resistors_SMD:R_0603_HandSoldering, F.Cu at (123.0, 73.0)
- added R13: 100k, Resistors_SMD:R_0603_HandSoldering, F.Cu at (152.7, 65.6)
- added R14: 100k, Resistors_SMD:R_0603_HandSoldering, F.Cu at (124.0, 70.0)
- added R15: 1k, Resistors_SMD:R_0603_HandSoldering, F.Cu at (173.3, 104.7)
- added R16: 330, Resistors_SMD:R_0603_HandSoldering, F.Cu at (205.0, 60.9)
- added R17: 330, Resistors_SMD:R_0603_HandSoldering, F.Cu at (205.0, 63.9)
- added R18: 330, Resistors_SMD:R_0603_HandSoldering, F.Cu at (205.1, 66.8)
- added R19: 330, Resistors_SMD:R_0603_HandSoldering, F.Cu at (107.5, 57.0)
- added R2: 330, Resistors_SMD:R_0603_HandSoldering, F.Cu at (165.0, 58.0)
- added R3: 100k, Resistors_SMD:R_0603_HandSoldering, F.Cu at (165.0, 60.0)
- added R4: 330, Resistors_SMD:R_0603_HandSoldering, F.Cu at (159.7, 63.9)
- added R5: 100k, Resistors_SMD:R_0603_HandSoldering, F.Cu at (162.4, 62.7)
- added R6: 10k, Resistors_SMD:R_0603_HandSoldering, F.Cu at (138.1, 79.0)
- added R7: 100k, Resistors_SMD:R_0603_HandSoldering, F.Cu at (151.3, 67.3)
- added R8: 1k, Resistors_SMD:R_0603_HandSoldering, F.Cu at (116.0, 71.0)
- added R9: 100k, Resistors_SMD:R_0603_HandSoldering, F.Cu at (147.8, 65.2)
- added RV1: POT, Potentiometers:Potentiometer_Trimmer_ACP_CA6v_Horizontal, B.Cu at (131.1, 56.0)
- added SH1: ARDUINO_NANO, SHIELD_ARDUINO:ARDUINO_NANO_2_CONTOUR_ELL, B.Cu at (235.1, 71.6)
- added SW1: Rotary_Encoder_Switch, bilge-alarm-parts:Encoder_Bourns_PEC12R-4xxxF-Sxxxx, F.Cu at (197.7, 80.6)
- added SW2: SW_SPST, Buttons_Switches_SMD:SW_SPST_EVPBF, F.Cu at (107.5, 81.0)
- added U1: 74HC595, Housings_SOIC:SOIC-16_3.9x9.9mm_Pitch1.27mm, F.Cu at (151.0, 60.0)
- added U2: LM7805CT, TO_SOT_Packages_THT:TO-220_Vertical, B.Cu at (139.9, 74.7)
- added U3: SP3481CN, Housings_SOIC:SOIC-8_3.9x4.9mm_Pitch1.27mm, F.Cu at (179.8, 104.2)
Routing:
- net +5V: track 0.00 -> 61.5 mm
- net Net-(C10-Pad1): track 0.00 -> 61.3 mm
- net Net-(DS1-Pad4): track 0.00 -> 29.1 mm
- net Net-(R2-Pad2): track 0.00 -> 23.9 mm, vias 0 -> 2
- net Net-(DS1-Pad6): track 0.00 -> 21.4 mm
- net +12V: track 0.00 -> 14.1 mm
- net GND: track 0.00 -> 9.09 mm, vias 0 -> 3
- net Net-(LS1-Pad2): track 0.00 -> 7.17 mm
- net Net-(DS1-Pad14): track 0.00 -> 5.80 mm
- net Net-(DS1-Pad13): track 0.00 -> 5.27 mm
- net Net-(DS1-Pad12): track 0.00 -> 4.74 mm
- net /LATCH: track 0.00 -> 4.67 mm
- net Net-(DS1-Pad11): track 0.00 -> 4.38 mm
- net Net-(DS1-Pad16): track 0.00 -> 3.61 mm
- net /DATA: track 0.00 -> 3.27 mm
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Other:
- board outline added: 115 x 45 mm
